File: eagle/NJM13700_MCP4922_DCA/NJM13700_MCP4922_DCA.brd (EAGLE design)
At the start: 100 x 80 mm, 38 parts, among them IC1 LM13600AN, IC2 MCP4922, IC3 TL072, IC4 TA480335, T1 2SA1015

Commit message: change parameters
Connections:
- net AGND: now also IC1.13, IC1.3; no longer IC1.14, IC1.4
- net N$10: now also IC3.6; no longer IC3.2
- net N$12: now also IC1.16; no longer IC1.1
- net N$14: now also IC1.4, IC1.5, IC1.7; no longer IC1.10, IC1.12, IC1.13
- net N$16: now also IC3.1, IC3.2; no longer IC3.6, IC3.7
- net N$4: now also IC1.14; no longer IC1.3
- net N$5: now also IC1.10, IC1.12; no longer IC1.5, IC1.7
- net N$6: now also IC1.9; no longer IC1.8
- net N$9: now also IC3.7; no longer IC3.1
Changed lines of the file:
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@@
 <contactref element="R1" pad="A"/>
 <contactref element="R3" pad="1"/>
-<contactref element="IC1" pad="4"/>
+<contactref element="IC1" pad="13"/>
 <contactref element="R4" pad="1"/>
 <contactref element="JP2" pad="2"/>
 <contactref element="IC2" pad="12"/>
 <contactref element="C3" pad="2"/>
+<contactref element="IC3" pad="5"/>
+<contactref element="R9" pad="1"/>
 <contactref element="IC3" pad="3"/>
-<contactref element="R9" pad="1"/>
-<contactref element="IC3" pad="5"/>
-<contactref element="IC1" pad="14"/>
+<contactref element="IC1" pad="3"/>
 <contactref element="C5" pad="1"/>
 <contactref element="C4" pad="2"/>
@@
 <wire x1="43.18" y1="33.02" x2="55.88" y2="35.56" width="0" layer="19" extent="1-1"/>
 <wire x1="38.1" y1="40.64" x2="43.18" y2="33.02" width="0" layer="19" extent="1-1"/>
-<wire x1="35.56" y1="43.18" x2="38.1" y2="40.64" width="0" layer="19" extent="1-1"/>
-<wire x1="33.02" y1="50.8" x2="35.56" y2="43.18" width="0" layer="19" extent="1-1"/>
-<wire x1="38.1" y1="53.34" x2="33.02" y2="50.8" width="0" layer="19" extent="1-1"/>
+<wire x1="35.56" y1="50.8" x2="38.1" y2="40.64" width="0" layer="19" extent="1-1"/>
+<wire x1="33.02" y1="43.18" x2="35.56" y2="50.8" width="0" layer="19" extent="1-1"/>
+<wire x1="38.1" y1="53.34" x2="33.02" y2="43.18" width="0" layer="19" extent="1-1"/>
 <wire x1="33.02" y1="33.02" x2="38.1" y2="40.64" width="0" layer="19" extent="1-1"/>
 <wire x1="20.32" y1="35.56" x2="33.02" y2="33.02" width="0" layer="19" extent="1-1"/>
@@
 <wire x1="20.32" y1="22.86" x2="20.32" y2="35.56" width="0" layer="19" extent="1-1"/>
 <wire x1="48.26" y1="20.32" x2="43.18" y2="33.02" width="0" layer="19" extent="1-1"/>
-<wire x1="48.26" y1="17.78" x2="48.26" y2="20.32" width="0" layer="19" extent="1-1"/>
-<wire x1="43.18" y1="15.24" x2="48.26" y2="17.78" width="0" layer="19" extent="1-1"/>
+<wire x1="45.72" y1="10.16" x2="48.26" y2="20.32" width="0" layer="19" extent="1-1"/>
+<wire x1="43.18" y1="15.24" x2="45.72" y2="10.16" width="0" layer="19" extent="1-1"/>
 <wire x1="45.72" y1="10.16" x2="43.18" y2="15.24" width="0" layer="19" extent="1-1"/>
-<wire x1="55.88" y1="12.7" x2="48.26" y2="17.78" width="0" layer="19" extent="1-1"/>
+<wire x1="55.88" y1="12.7" x2="45.72" y2="10.16" width="0" layer="19" extent="1-1"/>
 <wire x1="27.94" y1="10.16" x2="20.32" y2="22.86" width="0" layer="19" extent="1-1"/>
 <wire x1="27.94" y1="7.62" x2="27.94" y2="10.16" width="0" layer="19" extent="1-1"/>
@@
 <contactref element="R3" pad="2"/>
 <contactref element="C1" pad="-"/>
-<contactref element="IC1" pad="3"/>
-<wire x1="33.02" y1="40.64" x2="33.02" y2="43.18" width="0" layer="19" extent="1-1"/>
+<contactref element="IC1" pad="14"/>
+<wire x1="33.02" y1="40.64" x2="33.02" y2="50.8" width="0" layer="19" extent="1-1"/>
 <wire x1="30.48" y1="38.1" x2="33.02" y2="40.64" width="0" layer="19" extent="1-1"/>
 </signal>
 <signal name="N$5">
-<contactref element="IC1" pad="5"/>
-<contactref element="IC1" pad="7"/>
+<contactref element="IC1" pad="12"/>
+<contactref element="IC1" pad="10"/>
 <contactref element="R4" pad="2"/>
-<wire x1="43.18" y1="40.64" x2="43.18" y2="43.18" width="0" layer="19" extent="1-1"/>
-<wire x1="38.1" y1="43.18" x2="43.18" y2="43.18" width="0" layer="19" extent="1-1"/>
+<wire x1="43.18" y1="40.64" x2="43.18" y2="50.8" width="0" layer="19" extent="1-1"/>
+<wire x1="38.1" y1="50.8" x2="43.18" y2="50.8" width="0" layer="19" extent="1-1"/>
 </signal>
 <signal name="N$6">
-<contactref element="IC1" pad="8"/>
+<contactref element="IC1" pad="9"/>
 <contactref element="R5" pad="2"/>
 <contactref element="C2" pad="-"/>
-<wire x1="45.72" y1="43.18" x2="48.26" y2="43.18" width="0" layer="19" extent="1-1"/>
+<wire x1="45.72" y1="50.8" x2="48.26" y2="43.18" width="0" layer="19" extent="1-1"/>
 <wire x1="48.26" y1="40.64" x2="48.26" y2="43.18" width="0" layer="19" extent="1-1"/>
 </signal>
@@
 <signal name="N$10">
 <contactref element="R7" pad="1"/>
-<contactref element="IC3" pad="2"/>
+<contactref element="IC3" pad="6"/>
 <contactref element="R8" pad="2"/>
 <wire x1="50.8" y1="20.32" x2="53.34" y2="20.32" width="0" layer="19" extent="1-1"/>
-<wire x1="50.8" y1="17.78" x2="50.8" y2="20.32" width="0" layer="19" extent="1-1"/>
+<wire x1="48.26" y1="10.16" x2="50.8" y2="20.32" width="0" layer="19" extent="1-1"/>
 </signal>
 <signal name="N$9">
-<contactref element="IC3" pad="1"/>
+<contactref element="IC3" pad="7"/>
 <contactref element="T1" pad="B"/>
-<wire x1="38.1" y1="27.94" x2="53.34" y2="17.78" width="0" layer="19" extent="1-1"/>
+<wire x1="38.1" y1="27.94" x2="50.8" y2="10.16" width="0" layer="19" extent="1-1"/>
 </signal>
 <signal name="N$11">
@@
 </signal>
 <signal name="N$12">
-<contactref element="IC1" pad="1"/>
+<contactref element="IC1" pad="16"/>
 <contactref element="T1" pad="C"/>
-<wire x1="40.64" y1="27.94" x2="27.94" y2="43.18" width="0" layer="19" extent="1-1"/>
+<wire x1="40.64" y1="27.94" x2="27.94" y2="50.8" width="0" layer="19" extent="1-1"/>
 </signal>
 <signal name="N$16">
-<contactref element="IC3" pad="6"/>
-<contactref element="IC3" pad="7"/>
-<wire x1="48.26" y1="10.16" x2="50.8" y2="10.16" width="0" layer="19" extent="1-1"/>
+<contactref element="IC3" pad="2"/>
+<contactref element="IC3" pad="1"/>
+<wire x1="50.8" y1="17.78" x2="53.34" y2="17.78" width="0" layer="19" extent="1-1"/>
 </signal>
 <signal name="N$14">
-<contactref element="IC1" pad="13"/>
-<contactref element="IC1" pad="12"/>
-<contactref element="IC1" pad="10"/>
-<wire x1="38.1" y1="50.8" x2="43.18" y2="50.8" width="0" layer="19" extent="1-1"/>
-<wire x1="35.56" y1="50.8" x2="38.1" y2="50.8" width="0" layer="19" extent="1-1"/>
+<contactref element="IC1" pad="4"/>
+<contactref element="IC1" pad="5"/>
+<contactref element="IC1" pad="7"/>
+<wire x1="38.1" y1="43.18" x2="43.18" y2="43.18" width="0" layer="19" extent="1-1"/>
+<wire x1="35.56" y1="43.18" x2="38.1" y2="43.18" width="0" layer="19" extent="1-1"/>
 </signal>
 <signal name="+5V">

Commit message: Add: Board design
Parts:
- added RCA1, RCA2: ATD_RCA_JACK-DIP, mylib2:ATD_RCA_JACK_DIP
- C10, C12, C8: device rcl:E2,5-6 -> rcl:E5-8,5
- C3: device rcl:C050-025X075 -> rcl:C050-024X044
- moved C6 45.4 mm to (35.6, 52.1)
- moved C7 45.4 mm to (22.9, 57.1)
- moved IC3 45.4 mm to (29.2, 54.6)
- moved C8 33.3 mm to (58.4, 17.8), turned to 180 degrees
- moved R7 30.7 mm to (31.8, 48.3), turned to 0 degrees
- moved JP2 30.6 mm to (88.9, 39.4)
- moved R8 30.5 mm to (31.8, 45.7), turned to 180 degrees
- moved TP1 28.4 mm to (2.54, 25.4)
- moved C12 25.1 mm to (73.7, 22.9), turned to 180 degrees
- moved C13 24.7 mm to (16.5, 15.2)
- moved D1 24.3 mm to (59.7, 25.4)
- moved C2 21.7 mm to (69.8, 50.8)
- moved C11 21.3 mm to (63.5, 34.3), turned to 90 degrees
- moved T1 20.3 mm to (40.6, 48.3), turned to 90 degrees
- moved C5 20.1 mm to (58.4, 47.0), turned to 90 degrees
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Connections:
- net AGND: now also IC1.14, IC1.4, RCA1.P$2, RCA2.P$2; no longer IC1.13, IC1.3
- net N$1: now also RCA1.P$1
- net N$12: now also IC1.1; no longer IC1.16
- net N$14: now also IC1.10, IC1.12, IC1.13; no longer IC1.4, IC1.5, IC1.7
- net N$17: now also RCA2.P$1
- net N$4: now also IC1.3; no longer IC1.14
- net N$5: now also IC1.5, IC1.7; no longer IC1.10, IC1.12
- net N$6: now also IC1.8; no longer IC1.9
Other:
- board size 100 x 80 mm -> 93.7 x 71.1 mm

Commit message: updated schematic & board designe
Parts:
- added LED1, LED2: Green, led:LED3MM
- added R10, R11: 1k, rcl:0207/7
- C1: device rcl:E2,5-6 -> rcl:E5-6
- IC4: value TA480335 -> TA48M033F
- JP4: value PIN -> (none); device pinhead:1X03 -> pinhead:1X04
- R4: value 33k -> 27k
- TP1: value TPB1,27 -> TPPAD1-13; device testpad:B1,27 -> testpad:P1-13
- moved C8 5.68 mm to (63.5, 20.3), turned to 0 degrees
- moved JP5 5.08 mm to (27.9, 15.2)
- moved JP6 5.08 mm to (27.9, 12.7)
- moved TP1 3.59 mm to (5.08, 22.9)
- moved JP4 2.84 mm to (78.7, 8.89), turned to 90 degrees
- moved JP1 2.54 mm to (5.08, 39.4)
- moved C3 2.54 mm to (48.3, 25.4)
- moved C4 2.54 mm to (57.1, 63.5)
- moved C5 2.54 mm to (58.4, 49.5)
- moved C6 2.54 mm to (35.6, 54.6)
- moved C7 2.54 mm to (22.9, 59.7)
- moved IC1 2.54 mm to (54.6, 57.1)
- moved IC3 2.54 mm to (29.2, 57.1)
- moved JP3 2.54 mm to (27.9, 10.2)
- moved R4 2.54 mm to (55.9, 47.0)
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Connections:
- new net N$15: LED2.A, R11.1
- new net N$18: LED1.A, R10.1
- net +5V: now also R10.2
- net -5V: now also JP4.4, LED2.K; no longer JP4.3
- net AGND: now also JP4.3, LED1.K, R11.2, RCA1.P$5, RCA1.P$6, RCA1.P$7, RCA1.P$8, RCA2.P$5, RCA2.P$6, RCA2.P$7, RCA2.P$8; no longer RCA1.P$2, RCA2.P$2
- net N$1: now also RCA1.P$2, RCA1.P$3, RCA1.P$4
- net N$17: now also RCA2.P$2, RCA2.P$3, RCA2.P$4
Routing:
- net AGND: track 0.00 -> 391.5 mm
- net +5V: track 0.00 -> 118.4 mm
- net -5V: track 0.00 -> 115.5 mm
- net +3V3: track 0.00 -> 108.8 mm
- net N$17: track 0.00 -> 43.2 mm
- net N$8: track 0.00 -> 41.7 mm
- net N$7: track 0.00 -> 35.6 mm
- net N$1: track 0.00 -> 35.6 mm
- net N$4: track 0.00 -> 17.3 mm
- net !LDAC: track 0.00 -> 17.3 mm
- net N$9: track 0.00 -> 12.7 mm
- net N$13: track 0.00 -> 12.7 mm
- net N$5: track 0.00 -> 12.7 mm
- net N$14: track 0.00 -> 12.7 mm
- net N$3: track 0.00 -> 10.2 mm
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
Commit message: IC1、IC2の電源ラインのGNDへの接続を消去
Parts:
- JP4: value (none) -> PWR_IN
Changed lines of the file:
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@@
 <element name="RCA1" library="mylib2" package="ATD_RCA_JACK_DIP" value="ATD_RCA_JACK-DIP" x="7.62" y="52.07"/>
 <element name="RCA2" library="mylib2" package="ATD_RCA_JACK_DIP" value="ATD_RCA_JACK-DIP" x="86.36" y="52.07" rot="R180"/>
-<element name="JP4" library="pinhead" package="1X04" value="" x="78.74" y="8.89" rot="R90"/>
+<element name="JP4" library="pinhead" package="1X04" value="PWR_IN" x="78.74" y="8.89" rot="R90"/>
 <element name="LED1" library="led" package="LED3MM" value="Green" x="83.82" y="8.89" rot="R90"/>
 <element name="LED2" library="led" package="LED3MM" value="Green" x="83.82" y="16.51" rot="R90"/>

Commit message: Update: board design
Parts:
- moved R6 23.4 mm to (20.3, 27.9), turned to 180 degrees
- moved C3 23.0 mm to (25.4, 27.9), turned to 270 degrees
- moved IC2 12.7 mm to (38.1, 21.6)
- moved C13 12.7 mm to (29.2, 15.2)
- moved JP3 12.7 mm to (40.6, 10.2)
- moved JP5 12.7 mm to (40.6, 15.2)
- moved JP6 12.7 mm to (40.6, 12.7)
Routing:
- net N$7: track 35.6 -> 10.2 mm
- net +3V3: track 108.8 -> 91.0 mm
- net N$8: track 41.7 -> 58.0 mm
- net AGND: track 391.5 -> 401.7 mm
